Commit message: Keep the active short-arm Mojia recipe and remove obsolete training artifacts

File: assets/robots/mojia/urdf/robot.urdf (robot description, URDF)
Before this commit: robot mojia_v3_8, 24 links, 23 joints
Links:
- link left_elbow_yaw: mass 0.8163 -> 0.6663; geometry collision mesh filename=../meshes/left_elbow_yaw.STL; visual mesh filename=../meshes/left_elbow_yaw.STL
- link right_elbow_yaw: mass 0.8163 -> 0.6663; geometry collision mesh filename=../meshes/right_elbow_yaw.STL; visual mesh filename=../meshes/right_elbow_yaw.STL
